Commit message: feat: integrate Gazebo differential-drive control

File: src/ai_robot_description/urdf/ai_robot.urdf.xacro (robot description, xacro)
@@ -1,4 +1,5 @@
 <?xml version="1.0"?>
 <robot xmlns:xacro="http://www.ros.org/wiki/xacro" name="ai_robot">
+  <xacro:arg name="controllers_file" default=""/>
   <xacro:property name="base_length" value="0.42"/>
   <xacro:property name="base_width" value="0.30"/>
@@ -75,3 +76,20 @@
     <parent link="base_link"/><child link="sensor_link"/><origin xyz="0.10 0 0.10"/>
   </joint>
+  <ros2_control name="GazeboSimSystem" type="system">
+    <hardware><plugin>gz_ros2_control/GazeboSimSystem</plugin></hardware>
+    <joint name="left_wheel_joint">
+      <command_interface name="velocity"><param name="min">-8.0</param><param name="max">8.0</param></command_interface>
+      <state_interface name="position"/><state_interface name="velocity"/>
+    </joint>
+    <joint name="right_wheel_joint">
+      <command_interface name="velocity"><param name="min">-8.0</param><param name="max">8.0</param></command_interface>
+      <state_interface name="position"/><state_interface name="velocity"/>
+    </joint>
+  </ros2_control>
+  <gazebo>
+    <plugin filename="libgz_ros2_control-system.so"
+            name="gz_ros2_control::GazeboSimROS2ControlPlugin">
+      <parameters>$(arg controllers_file)</parameters>
+    </plugin>
+  </gazebo>
 </robot>

Commit message: feat: define M3 sensor frames

File: src/ai_robot_description/urdf/ai_robot.urdf.xacro (robot description, xacro)
@@ -71,8 +71,27 @@
     <parent link="base_link"/><child link="caster_link"/><origin xyz="-0.15 0 -0.04"/>
   </joint>
-  <!-- M2 reserves one generic sensor mounting frame; sensors are introduced in M3. -->
+  <!-- Generic sensor mounting datum retained as the parent of M3 sensor frames. -->
   <link name="sensor_link"/>
   <joint name="sensor_joint" type="fixed">
     <parent link="base_link"/><child link="sensor_link"/><origin xyz="0.10 0 0.10"/>
+  </joint>
+  <!-- M3 frozen simulated sensor extrinsics; REP-103 body axes: x forward, y left, z up. -->
+  <link name="laser_link"/>
+  <joint name="laser_joint" type="fixed">
+    <parent link="sensor_link"/><child link="laser_link"/><origin xyz="0 0 0.06" rpy="0 0 0"/>
+  </joint>
+  <link name="camera_link"/>
+  <joint name="camera_joint" type="fixed">
+    <parent link="sensor_link"/><child link="camera_link"/><origin xyz="0.08 0 0.02" rpy="0 0 0"/>
+  </joint>
+  <!-- Optical convention: z forward, x right, y down. -->
+  <link name="camera_optical_link"/>
+  <joint name="camera_optical_joint" type="fixed">
+    <parent link="camera_link"/><child link="camera_optical_link"/>
+    <origin xyz="0 0 0" rpy="-1.57079632679 0 -1.57079632679"/>
+  </joint>
+  <link name="imu_link"/>
+  <joint name="imu_joint" type="fixed">
+    <parent link="sensor_link"/><child link="imu_link"/><origin xyz="0 0 0" rpy="0 0 0"/>
   </joint>
   <ros2_control name="GazeboSimSystem" type="system">

Commit message: fix: align M5 base footprint TF

File: src/ai_robot_description/urdf/ai_robot.urdf.xacro (robot description, xacro)
@@ -49,7 +49,7 @@
   <link name="base_footprint"/>
   <joint name="base_footprint_joint" type="fixed">
-    <parent link="base_footprint"/>
-    <child link="base_link"/>
-    <origin xyz="0 0 ${wheel_radius}"/>
+    <parent link="base_link"/>
+    <child link="base_footprint"/>
+    <origin xyz="0 0 ${-wheel_radius}"/>
   </joint>
   <link name="base_link">
